File: Electrical/ESP32-S3-Expansion.kicad_sch (KiCad schematic)
At the start: 17 parts, among them CN1 1.0T-4PLTPZ, J1 Conn_01x04, P1 USB_C_Plug_USB2.0, SW1 TS-1088-AR02016, SW2 TS-1088-AR02016, U1 ESP32-S3-MINI-1-N4R2

Commit message: Restructured Schematic
Removed Borders
Changed Symbol of ESP32-S3
Changed Symbol of AP2112K-3.3
Parts:
- removed C?: 22uF, Capacitor_SMD:C_0603_1608Metric, symbol Device:C
- removed C? (x2): 1uF, Capacitor_SMD:C_0603_1608Metric, symbol Device:C
- removed C? (x2): 100nF, Capacitor_SMD:C_0402_1005Metric, symbol Device:C
- removed J1: Conn_01x04, Connector_PinHeader_2.54mm:PinHeader_1x04_P2.54mm_Vertical, symbol Connector_Generic:Conn_01x04
- removed LED?: WS2812B-2020, _mykicadlib:LED-SMD_4P-L2.0-W2.0-TL_WS2812B-2020, symbol _mykicadlib:WS2812B-2020
- removed R?: 10K, Resistor_SMD:R_0402_1005Metric, symbol Device:R
- removed SW1, SW2: TS-1088-AR02016, _mykicadlib:SW-SMD_L3.9-W3.0-P4.45, symbol _mykicadlib:SW_TS-1088-AR02016
- removed U1: ESP32-S3-MINI-1-N4R2, _mykicadlib:ESP32-S3-MINI-1-N4R2, symbol _mykicadlib:ESP32-S3-MINI-1-N4R2
- removed U?: AP2112K-3.3TRG1, _mykicadlib:SOT-25-5_AP2112K, symbol _mykicadlib:AP2112K-3.3TRG1
- added C1, C2: 10uF, Capacitor_SMD:C_0201_0603Metric_Pad0.64x0.40mm_HandSolder, symbol Device:C_Small
- added C?: 100nF, Capacitor_SMD:C_0402_1005Metric, symbol Device:C
- added C?: 22uF, Capacitor_SMD:C_0603_1608Metric, symbol Device:C
- added J1: Conn_01x06, symbol Connector_Generic:Conn_01x06
- added LED?: WS2812B-2020, _mykicadlib:LED-SMD_4P-L2.0-W2.0-TL_WS2812B-2020, symbol _mykicadlib:WS2812B-2020
- added U1: AP2112K-3.3, Package_TO_SOT_SMD:SOT-23-5, symbol Regulator_Linear:AP2112K-3.3
- added U2: SN65HVD230, Package_SO:SOIC-8_3.9x4.9mm_P1.27mm, symbol Interface_CAN_LIN:SN65HVD230
- added U3: ESP32-S3, Espressif:ESP32-S3-MINI-1, symbol Espressif:ESP32-S3
Connections:
- net +3V3: now also C2.1, C?.1, C?.1, LED?.4 (VDD), U1.5 (VOUT), U2.3 (VCC)
- net D+: now also U3.26 (GPIO20/USB_D+/ADC2_CH9)
- net D-: now also U3.25 (GPIO19/USB_D-/ADC2_CH8)
- net GND: now also C1.2, C2.2, C?.2, C?.2, J1.4 (Pin_4), LED?.2 (GND), U1.2 (GND), U2.2 (GND), U3.57 (GND)
- net NPXL: now also LED?.3 (DI), U3.42 (GPIO37)
- net RXD0: now also J1.3 (Pin_3), U3.50 (U0RXD/PROG/GPIO44)
- net SCL: now also U3.7 (GPIO2/ADC1_CH1)
- net SDA: now also U3.8 (GPIO3/ADC1_CH2)
- net TXD0: now also J1.2 (Pin_2), U3.49 (U0TXD/PROG/GPIO43)
- new net +3.3V: U3.2 (VDD3P3), U3.20 (VDD3P3_RTC), U3.29 (VDD_SPI), U3.3 (VDD3P3), U3.46 (VDD3P3_CPU), U3.55 (VDDA), U3.56 (VDDA)
- new net CAN_H: J1.5 (Pin_5), U2.7 (CANH)
- new net CAN_L: J1.6 (Pin_6), U2.6 (CANL)
- new net CAN_RX: U2.4 (R), U3.10 (GPIO5/ADC1_CH4)
- new net CAN_TX: U2.1 (D), U3.9 (GPIO4/ADC1_CH3)
- new net VBUS: C1.1, J1.1 (Pin_1), U1.1 (VIN), U1.3 (EN)
- no-connect marks 36 -> 43
Other:
- note added: "5V to 3.3V 600mA"
- note added: "CAN Transceiver"
- note added: "Power Cap"
- note removed: "3.3V LDO"
- note removed: "Boot Switch"
- note removed: "ESP"
- note removed: "ESP Power Caps"
- note removed: "Programming Pins"
- note removed: "Reset Switch"
- moved on the sheet: CN1, H1, H2, P1, R1
