File: Electrical/ESP32-S3-Expansion.kicad_pcb (KiCad board)
At the start: 2 copper layers, 26 x 28 mm, 22 parts, among them CN1 1.0T-4PLTPZ, P1 USB_C_Plug_USB2.0, SW1 TS-1088-AR02016, SW2 TS-1088-AR02016, U1 AP2112K-3.3TRG1, U2 ESP32-S3-MINI-1-N4R2

Commit message: Cleared PCB
Parts:
- removed C1, C2: 1uF, Capacitor_SMD:C_0603_1608Metric
- removed C3: 22uF, Capacitor_SMD:C_0603_1608Metric
- removed C4, C5: 100nF, Capacitor_SMD:C_0402_1005Metric
- removed CN1: 1.0T-4PLTPZ, _mykicadlib:FPC-SMD_4P-P1.00_1.0T-4PLTPZ
- removed G***: LOGO, artwork:spacehuhn_logo_text_small
- removed G1: LOGO, artwork:spacehuhn_logo_text_big-mask
- removed G2: LOGO, artwork:star_small
- removed G3, G4: LOGO, artwork:star_tiny
- removed G5: LOGO, artwork:oshw_logo_small
- removed H1, H2: MountingHole, MountingHole:MountingHole_2.2mm_M2
- removed LED1: WS2812B-2020, _mykicadlib:LED-SMD_4P-L2.0-W2.0-TL_WS2812B-2020
- removed R1: 5.1k, Resistor_SMD:R_0402_1005Metric
- removed R2: 10K, Resistor_SMD:R_0402_1005Metric
- removed SW1, SW2: TS-1088-AR02016, _mykicadlib:SW-SMD_L3.9-W3.0-P4.45
- removed U1: AP2112K-3.3TRG1, _mykicadlib:SOT-25-5_AP2112K
- removed U2: ESP32-S3-MINI-1-N4R2, _mykicadlib:ESP32-S3-MINI-1-N4R2
Routing:
- net +3V3: track 52.1 -> 0.00 mm, vias 2 -> 0
- net /RESET: track 24.2 -> 0.00 mm, vias 2 -> 0
- net +5V: track 22.7 -> 0.00 mm
- net /BOOT: track 19.2 -> 0.00 mm
- net /SDA: track 18.7 -> 0.00 mm
- net /SCL: track 18.5 -> 0.00 mm
- net GND: track 12.1 -> 0.00 mm, vias 12 -> 0
- net /NPXL: track 8.56 -> 0.00 mm, vias 2 -> 0
- net /D+: track 4.61 -> 0.00 mm
- net /D-: track 4.46 -> 0.00 mm
- net Net-(P1-CC): track 3.12 -> 0.00 mm
- removed copper zone on B.Cu, net GND
- removed copper zone on F.Cu, net GND
Other:
- board text removed: "BOOT"
- board text removed: "Framework ESP32-S3"
- board text removed: "RST"
